File: cad/board/controller_board.sch (KiCad schematic (older format))
At the start: 13 parts, among them J1 Barrel_Jack, J2 Conn_01x12, J3 Conn_01x16, J4 Conn_01x12, U2 DIP-16-Socket

Commit message: better layout, gcode
Parts:
- R1, R2, R3, R4: footprint Resistors_ThroughHole:R_Axial_DIN0207_L6.3mm_D2.5mm_P15.24mm_Horizontal -> Resistors_SMD:R_1206_HandSoldering
Changed lines of the file:
@@
 F 0 "R1" V 5101 1369 50  0000 C CNN
 F 1 "R" V 5021 1369 50  0000 C CNN
-F 2 "Resistors_ThroughHole:R_Axial_DIN0207_L6.3mm_D2.5mm_P15.24mm_Horizontal" V 4951 1369 50  0001 C CNN
+F 2 "Resistors_SMD:R_1206_HandSoldering" V 4951 1369 50  0001 C CNN
 F 3 "" H 5021 1369 50  0001 C CNN
 	1    5021 1369
@@
 F 0 "R2" V 5101 1669 50  0000 C CNN
 F 1 "R" V 5021 1669 50  0000 C CNN
-F 2 "Resistors_ThroughHole:R_Axial_DIN0207_L6.3mm_D2.5mm_P15.24mm_Horizontal" V 4951 1669 50  0001 C CNN
+F 2 "Resistors_SMD:R_1206_HandSoldering" V 4951 1669 50  0001 C CNN
 F 3 "" H 5021 1669 50  0001 C CNN
 	1    5021 1669
@@
 F 0 "R3" V 5101 1969 50  0000 C CNN
 F 1 "R" V 5021 1969 50  0000 C CNN
-F 2 "Resistors_ThroughHole:R_Axial_DIN0207_L6.3mm_D2.5mm_P15.24mm_Horizontal" V 4951 1969 50  0001 C CNN
+F 2 "Resistors_SMD:R_1206_HandSoldering" V 4951 1969 50  0001 C CNN
 F 3 "" H 5021 1969 50  0001 C CNN
 	1    5021 1969
@@
 F 0 "R4" V 5101 2269 50  0000 C CNN
 F 1 "R" V 5021 2269 50  0000 C CNN
-F 2 "Resistors_ThroughHole:R_Axial_DIN0207_L6.3mm_D2.5mm_P15.24mm_Horizontal" V 4951 2269 50  0001 C CNN
+F 2 "Resistors_SMD:R_1206_HandSoldering" V 4951 2269 50  0001 C CNN
 F 3 "" H 5021 2269 50  0001 C CNN
 	1    5021 2269
@@
 NoConn ~ 7784 1915
 $Comp
-L VCC #PWR?
+L VCC #PWR025
 U 1 1 5A171CF0
 P 6356 2088
-F 0 "#PWR?" H 6356 1938 50  0001 C CNN
+F 0 "#PWR025" H 6356 1938 50  0001 C CNN
 F 1 "VCC" V 6354 2272 50  0000 C CNN
 F 2 "" H 6356 2088 50  0001 C CNN
@@
 $EndComp
 $Comp
-L VCC #PWR?
+L VCC #PWR026
 U 1 1 5A171D56
 P 6359 2488
-F 0 "#PWR?" H 6359 2338 50  0001 C CNN
+F 0 "#PWR026" H 6359 2338 50  0001 C CNN
 F 1 "VCC" V 6357 2672 50  0000 C CNN
 F 2 "" H 6359 2488 50  0001 C CNN
@@
 $EndComp
 $Comp
-L VCC #PWR?
+L VCC #PWR027
 U 1 1 5A171E24
 P 6361 2900
-F 0 "#PWR?" H 6361 2750 50  0001 C CNN
+F 0 "#PWR027" H 6361 2750 50  0001 C CNN
 F 1 "VCC" V 6359 3084 50  0000 C CNN
 F 2 "" H 6361 2900 50  0001 C CNN
@@
 $EndComp
 $Comp
-L GND #PWR?
+L GND #PWR028
 U 1 1 5A17208F
 P 6356 1788
-F 0 "#PWR?" H 6356 1538 50  0001 C CNN
+F 0 "#PWR028" H 6356 1538 50  0001 C CNN
 F 1 "GND" V 6355 1607 50  0000 C CNN
 F 2 "" H 6356 1788 50  0001 C CNN
@@
 $EndComp
 $Comp
-L GND #PWR?
+L GND #PWR029
 U 1 1 5A172129
 P 6359 2188
-F 0 "#PWR?" H 6359 1938 50  0001 C CNN
+F 0 "#PWR029" H 6359 1938 50  0001 C CNN
 F 1 "GND" V 6358 2007 50  0000 C CNN
 F 2 "" H 6359 2188 50  0001 C CNN
@@
 $EndComp
 $Comp
-L GND #PWR?
+L GND #PWR030
 U 1 1 5A172252
 P 6361 2600
-F 0 "#PWR?" H 6361 2350 50  0001 C CNN
+F 0 "#PWR030" H 6361 2350 50  0001 C CNN
 F 1 "GND" V 6360 2419 50  0000 C CNN
 F 2 "" H 6361 2600 50  0001 C CNN

Commit message: dunno
Parts:
- R1, R2, R3, R4: footprint Resistors_SMD:R_1206_HandSoldering -> Resistors_ThroughHole:R_Axial_DIN0309_L9.0mm_D3.2mm_P5.08mm_Vertical
Changed lines of the file:
@@
 F 0 "R1" V 5101 1369 50  0000 C CNN
 F 1 "R" V 5021 1369 50  0000 C CNN
-F 2 "Resistors_SMD:R_1206_HandSoldering" V 4951 1369 50  0001 C CNN
+F 2 "Resistors_ThroughHole:R_Axial_DIN0309_L9.0mm_D3.2mm_P5.08mm_Vertical" V 4951 1369 50  0001 C CNN
 F 3 "" H 5021 1369 50  0001 C CNN
 	1    5021 1369
@@
 F 0 "R2" V 5101 1669 50  0000 C CNN
 F 1 "R" V 5021 1669 50  0000 C CNN
-F 2 "Resistors_SMD:R_1206_HandSoldering" V 4951 1669 50  0001 C CNN
+F 2 "Resistors_ThroughHole:R_Axial_DIN0309_L9.0mm_D3.2mm_P5.08mm_Vertical" V 4951 1669 50  0001 C CNN
 F 3 "" H 5021 1669 50  0001 C CNN
 	1    5021 1669
@@
 F 0 "R3" V 5101 1969 50  0000 C CNN
 F 1 "R" V 5021 1969 50  0000 C CNN
-F 2 "Resistors_SMD:R_1206_HandSoldering" V 4951 1969 50  0001 C CNN
+F 2 "Resistors_ThroughHole:R_Axial_DIN0309_L9.0mm_D3.2mm_P5.08mm_Vertical" V 4951 1969 50  0001 C CNN
 F 3 "" H 5021 1969 50  0001 C CNN
 	1    5021 1969
@@
 F 0 "R4" V 5101 2269 50  0000 C CNN
 F 1 "R" V 5021 2269 50  0000 C CNN
-F 2 "Resistors_SMD:R_1206_HandSoldering" V 4951 2269 50  0001 C CNN
+F 2 "Resistors_ThroughHole:R_Axial_DIN0309_L9.0mm_D3.2mm_P5.08mm_Vertical" V 4951 2269 50  0001 C CNN
 F 3 "" H 5021 2269 50  0001 C CNN
 	1    5021 2269
